Commit message: Hand added to the arm

File: urdf/Igor_armed.urdf.xacro (robot description, xacro)
@@ -7,4 +7,5 @@
 	<xacro:include filename="$(find igor)/urdf/lowerleg.urdf.xacro" />
 	<xacro:include filename="$(find igor)/urdf/arm.urdf.xacro" />
+	<xacro:include filename="$(find igor)/urdf/my_hand.urdf.xacro" />
 	  <!-- Base Size -->
 	<xacro:property name="base_y_size" value="0.305" />
@@ -139,4 +140,8 @@
 		<origin xyz="${lower_leg_length + actuator_z_size/2.3} ${0} ${actuator_y_size/1.2}" rpy="${M_PI/2} ${0} 0" />
 	</xacro:igor_actuator>
+	<!--Hand-->
+	<xacro:my_hand prefix="Arm1" parent_link= "EndeffectorActuator">
+		<origin xyz="${0} ${0} ${0}" rpy="${0} ${0} ${0}" />
+	</xacro:my_hand>
 	<!--Robot Center Dummy-->
 	<link name="robot_center_link">

File: urdf/arm.urdf.xacro (robot description, xacro)
@@ -26,5 +26,5 @@
 			<parent link="${prefix}_armActuator"/>
 			<child  link="${prefix}_arm"/>
-			<limit effort="5" lower="${-2}" upper="${2}" velocity="10"/>
+			<limit effort="25" lower="${-2}" upper="${2}" velocity="10"/>
 			<axis xyz="0 0 1"/>
 			<dynamics damping="0.1"/>

Commit message: Pepsi can added in urdf

File: urdf/Igor_armed.urdf.xacro (robot description, xacro)
@@ -8,4 +8,5 @@
 	<xacro:include filename="$(find igor)/urdf/arm.urdf.xacro" />
 	<xacro:include filename="$(find igor)/urdf/my_hand.urdf.xacro" />
+	<xacro:include filename="$(find igor)/urdf/pepsi_can.urdf.xacro" />
 	  <!-- Base Size -->
 	<xacro:property name="base_y_size" value="0.305" />
@@ -144,4 +145,8 @@
 		<origin xyz="${0} ${0} ${0}" rpy="${0} ${0} ${0}" />
 	</xacro:my_hand>
+	<!--Pepsi Can  -->
+	<xacro:pepsi_can parent_link= "H1_base_link">
+		<origin xyz="${0.0} ${0} ${0.062}" rpy="${0} ${0} ${0}" />
+	</xacro:pepsi_can>
 	<!--Robot Center Dummy-->
 	<link name="robot_center_link">

File: urdf/my_hand.urdf.xacro (robot description, xacro)
@@ -43,5 +43,5 @@
 				<origin rpy="${0} ${0} ${0}" xyz="${0} ${0} ${0}"/>
 				<geometry>
-					<mesh filename="package://fh_desc/meshes/v2/palm_link_simple.dae" scale="0.5 0.5 0.5"/>
+					<mesh filename="package://igor/meshes/palm_link_simple.dae" scale="0.5 0.5 0.5"/>
 				</geometry>
 				<material name="light_grey">
@@ -52,5 +52,5 @@
 				<origin rpy="0 0 0" xyz="0 0 0"/>
 				<geometry>
-					<mesh filename="package://fh_desc/meshes/v2/palm_link_simple.dae" scale="0.5 0.5 0.5"/>
+					<mesh filename="package://igor/meshes/palm_link_simple.dae" scale="0.5 0.5 0.5"/>
 				</geometry>
 				<material name="light_grey">
@@ -100,5 +100,5 @@
 		      <origin rpy="0 0 0" xyz="0 0 0"/>
 		      <geometry>
-			<mesh filename="package://fh_desc/meshes/v2/finger_palm_link.dae" scale="0.5 0.5 0.5"/>
+			<mesh filename="package://igor/meshes/finger_palm_link.dae" scale="0.5 0.5 0.5"/>
 		      </geometry>
 		      <material name="light_grey">
@@ -121,14 +121,14 @@
 		      <origin rpy="0 0 0" xyz="0 0 0"/>
 		      <geometry>
-			<mesh filename="package://fh_desc/meshes/v2/finger_base_link_simple.dae" scale="0.5 0.5 0.5"/>
-		      </geometry>
-		      <material name="light_grey">
-			<color rgba="0.75 0.75 0.75 1.0"/>
-		      </material>
-		    </visual>
-		    <collision>
-		      <origin rpy="0 0 0" xyz="0 0 0"/>
-		      <geometry>
-			<mesh filename="package://fh_desc/meshes/v2/finger_base_link_simple.dae" scale="0.5 0.5 0.5"/>
+			<mesh filename="package://igor/meshes/finger_base_link_simple.dae" scale="0.5 0.5 0.5"/>
+		      </geometry>
+		      <material name="light_grey">
+			<color rgba="0.75 0.75 0.75 1.0"/>
+		      </material>
+		    </visual>
+		    <collision>
+		      <origin rpy="0 0 0" xyz="0 0 0"/>
+		      <geometry>
+			<mesh filename="package://igor/meshes/finger_base_link_simple.dae" scale="0.5 0.5 0.5"/>
 		      </geometry>
 		      <material name="light_grey">
@@ -146,14 +146,14 @@
 		      <origin rpy="0 0 0" xyz="0 0 0"/>
 		      <geometry>
-			<mesh filename="package://fh_desc/meshes/v2/finger_prox_link_simple.dae" scale="0.5 0.5 0.5"/>
-		      </geometry>
-		      <material name="light_grey">
-			<color rgba="0.75 0.75 0.75 1.0"/>
-		      </material>
-		    </visual>
-		    <collision>
-		      <origin rpy="0 0 0" xyz="0 0 0"/>
-		      <geometry>
-			<mesh filename="package://fh_desc/meshes/v2/finger_prox_link_simple.dae" scale="0.5 0.5 0.5"/>
+			<mesh filename="package://igor/meshes/finger_prox_link_simple.dae" scale="0.5 0.5 0.5"/>
+		      </geometry>
+		      <material name="light_grey">
+			<color rgba="0.75 0.75 0.75 1.0"/>
+		      </material>
+		    </visual>
+		    <collision>
+		      <origin rpy="0 0 0" xyz="0 0 0"/>
+		      <geometry>
+			<mesh filename="package://igor/meshes/finger_prox_link_simple.dae" scale="0.5 0.5 0.5"/>
 		      </geometry>
 		      <material name="light_grey">
@@ -171,14 +171,14 @@
 		      <origin rpy="0 0 0" xyz="0 0 0"/>
 		      <geometry>
-			<mesh filename="package://fh_desc/meshes/v2/finger_dist_link_simple.dae" scale="0.5 0.5 0.5"/>
-		      </geometry>
-		      <material name="light_grey">
-			<color rgba="0.75 0.75 0.75 1.0"/>
-		      </material>
-		    </visual>
-		    <collision>
-		      <origin rpy="0 0 0" xyz="0 0 0"/>
-		      <geometry>
-			<mesh filename="package://fh_desc/meshes/v2/finger_dist_link_simple.dae" scale="0.5 0.5 0.5"/>
+			<mesh filename="package://igor/meshes/finger_dist_link_simple.dae" scale="0.5 0.5 0.5"/>
+		      </geometry>
+		      <material name="light_grey">
+			<color rgba="0.75 0.75 0.75 1.0"/>
+		      </material>
+		    </visual>
+		    <collision>
+		      <origin rpy="0 0 0" xyz="0 0 0"/>
+		      <geometry>
+			<mesh filename="package://igor/meshes/finger_dist_link_simple.dae" scale="0.5 0.5 0.5"/>
 		      </geometry>
 		      <material name="light_grey">
@@ -253,14 +253,14 @@
 		      <origin rpy="0 0 0" xyz="0 0 0"/>
 		      <geometry>
-			<mesh filename="package://fh_desc/meshes/omd-d18-tip.dae" scale="0.5 0.5 0.5"/>
-		      </geometry>
-		      <material name="light_grey">
-			<color rgba="0.75 0.75 0.75 1.0"/>
-		      </material>
-		    </visual>
-		    <collision>
-		      <origin rpy="0 0 0" xyz="0 0 0"/>
-		      <geometry>
-			<mesh filename="package://fh_desc/meshes/omd-d18-tip.dae" scale="0.5 0.5 0.5"/>
+			<mesh filename="package://igor/meshes/omd-d18-tip.dae" scale="0.5 0.5 0.5"/>
+		      </geometry>
+		      <material name="light_grey">
+			<color rgba="0.75 0.75 0.75 1.0"/>
+		      </material>
+		    </visual>
+		    <collision>
+		      <origin rpy="0 0 0" xyz="0 0 0"/>
+		      <geometry>
+			<mesh filename="package://igor/meshes/omd-d18-tip.dae" scale="0.5 0.5 0.5"/>
 		      </geometry>
 		      <material name="light_grey">
@@ -288,5 +288,5 @@
 		      <origin rpy="0 0 0" xyz="0 0 0"/>
 		      <geometry>
-			<mesh filename="package://fh_desc/meshes/v2/finger_palm_link.dae" scale="0.5 0.5 0.5"/>
+			<mesh filename="package://igor/meshes/finger_palm_link.dae" scale="0.5 0.5 0.5"/>
 		      </geometry>
 		      <material name="light_grey">
@@ -309,14 +309,14 @@
 		      <origin rpy="0 0 0" xyz="0 0 0"/>
 		      <geometry>
-			<mesh filename="package://fh_desc/meshes/v2/finger_base_link_simple.dae" scale="0.5 0.5 0.5"/>
-		      </geometry>
-		      <material name="light_grey">
-			<color rgba="0.75 0.75 0.75 1.0"/>
-		      </material>
-		    </visual>
-		    <collision>
-		      <origin rpy="0 0 0" xyz="0 0 0"/>
-		      <geometry>
-			<mesh filename="package://fh_desc/meshes/v2/finger_base_link_simple.dae" scale="0.5 0.5 0.5"/>
+			<mesh filename="package://igor/meshes/finger_base_link_simple.dae" scale="0.5 0.5 0.5"/>
+		      </geometry>
+		      <material name="light_grey">
+			<color rgba="0.75 0.75 0.75 1.0"/>
+		      </material>
+		    </visual>
+		    <collision>
+		      <origin rpy="0 0 0" xyz="0 0 0"/>
+		      <geometry>
+			<mesh filename="package://igor/meshes/finger_base_link_simple.dae" scale="0.5 0.5 0.5"/>
 		      </geometry>
 		      <material name="light_grey">
@@ -334,14 +334,14 @@
 		      <origin rpy="0 0 0" xyz="0 0 0"/>
 		      <geometry>
-			<mesh filename="package://fh_desc/meshes/v2/finger_prox_link_simple.dae" scale="0.5 0.5 0.5"/>
-		      </geometry>
-		      <material name="light_grey">
-			<color rgba="0.75 0.75 0.75 1.0"/>
-		      </material>
-		    </visual>
-		    <collision>
-		      <origin rpy="0 0 0" xyz="0 0 0"/>
-		      <geometry>
-			<mesh filename="package://fh_desc/meshes/v2/finger_prox_link_simple.dae" scale="0.5 0.5 0.5"/>
+			<mesh filename="package://igor/meshes/finger_prox_link_simple.dae" scale="0.5 0.5 0.5"/>
+		      </geometry>
+		      <material name="light_grey">
+			<color rgba="0.75 0.75 0.75 1.0"/>
+		      </material>
+		    </visual>
+		    <collision>
+		      <origin rpy="0 0 0" xyz="0 0 0"/>
+		      <geometry>
+			<mesh filename="package://igor/meshes/finger_prox_link_simple.dae" scale="0.5 0.5 0.5"/>
 		      </geometry>
 		      <material name="light_grey">
@@ -359,14 +359,14 @@
 		      <origin rpy="0 0 0" xyz="0 0 0"/>
 		      <geometry>
-			<mesh filename="package://fh_desc/meshes/v2/finger_dist_link_simple.dae" scale="0.5 0.5 0.5"/>
-		      </geometry>
-		      <material name="light_grey">
-			<color rgba="0.75 0.75 0.75 1.0"/>
-		      </material>
-		    </visual>
-		    <collision>
-		      <origin rpy="0 0 0" xyz="0 0 0"/>
-		      <geometry>
-			<mesh filename="package://fh_desc/meshes/v2/finger_dist_link_simple.dae" scale="0.5 0.5 0.5"/>
+			<mesh filename="package://igor/meshes/finger_dist_link_simple.dae" scale="0.5 0.5 0.5"/>
+		      </geometry>
+		      <material name="light_grey">
+			<color rgba="0.75 0.75 0.75 1.0"/>
+		      </material>
+		    </visual>
+		    <collision>
+		      <origin rpy="0 0 0" xyz="0 0 0"/>
+		      <geometry>
+			<mesh filename="package://igor/meshes/finger_dist_link_simple.dae" scale="0.5 0.5 0.5"/>
 		      </geometry>
 		      <material name="light_grey">
@@ -441,14 +441,14 @@
 		      <origin rpy="0 0 0" xyz="0 0 0"/>
 		      <geometry>
-			<mesh filename="package://fh_desc/meshes/omd-d18-tip.dae" scale="0.5 0.5 0.5"/>
-		      </geometry>
-		      <material name="light_grey">
-			<color rgba="0.75 0.75 0.75 1.0"/>
-		      </material>
-		    </visual>
-		    <collision>
-		      <origin rpy="0 0 0" xyz="0 0 0"/>
-		      <geometry>
-			<mesh filename="package://fh_desc/meshes/omd-d18-tip.dae" scale="0.5 0.5 0.5"/>
+			<mesh filename="package://igor/meshes/omd-d18-tip.dae" scale="0.5 0.5 0.5"/>
+		      </geometry>
+		      <material name="light_grey">
+			<color rgba="0.75 0.75 0.75 1.0"/>
+		      </material>
+		    </visual>
+		    <collision>
+		      <origin rpy="0 0 0" xyz="0 0 0"/>
+		      <geometry>
+			<mesh filename="package://igor/meshes/omd-d18-tip.dae" scale="0.5 0.5 0.5"/>
 		      </geometry>
 		      <material name="light_grey">
@@ -476,5 +476,5 @@
 		      <origin rpy="0 0 0" xyz="0 0 0"/>
 		      <geometry>
-			<mesh filename="package://fh_desc/meshes/v2/finger_palm_link.dae" scale="0.5 0.5 0.5"/>
+			<mesh filename="package://igor/meshes/finger_palm_link.dae" scale="0.5 0.5 0.5"/>
 		      </geometry>
 		      <material name="light_grey">
@@ -497,14 +497,14 @@
 		      <origin rpy="0 0 0" xyz="0 0 0"/>
 		      <geometry>
-			<mesh filename="package://fh_desc/meshes/v2/finger_base_link_simple.dae" scale="0.5 0.5 0.5"/>
-		      </geometry>
-		      <material name="light_grey">
-			<color rgba="0.75 0.75 0.75 1.0"/>
-		      </material>
-		    </visual>
-		    <collision>
-		      <origin rpy="0 0 0" xyz="0 0 0"/>
-		      <geometry>
-			<mesh filename="package://fh_desc/meshes/v2/finger_base_link_simple.dae" scale="0.5 0.5 0.5"/>
+			<mesh filename="package://igor/meshes/finger_base_link_simple.dae" scale="0.5 0.5 0.5"/>
+		      </geometry>
+		      <material name="light_grey">
+			<color rgba="0.75 0.75 0.75 1.0"/>
+		      </material>
+		    </visual>
+		    <collision>
+		      <origin rpy="0 0 0" xyz="0 0 0"/>
+		      <geometry>
+			<mesh filename="package://igor/meshes/finger_base_link_simple.dae" scale="0.5 0.5 0.5"/>
 		      </geometry>
 		      <material name="light_grey">
@@ -522,14 +522,14 @@
 		      <origin rpy="0 0 0" xyz="0 0 0"/>
 		      <geometry>
-			<mesh filename="package://fh_desc/meshes/v2/finger_prox_link_simple.dae" scale="0.5 0.5 0.5"/>
-		      </geometry>
-		      <material name="light_grey">
-			<color rgba="0.75 0.75 0.75 1.0"/>
-		      </material>
-		    </visual>
-		    <collision>
-		      <origin rpy="0 0 0" xyz="0 0 0"/>
-		      <geometry>
-			<mesh filename="package://fh_desc/meshes/v2/finger_prox_link_simple.dae" scale="0.5 0.5 0.5"/>
+			<mesh filename="package://igor/meshes/finger_prox_link_simple.dae" scale="0.5 0.5 0.5"/>
+		      </geometry>
+		      <material name="light_grey">
+			<color rgba="0.75 0.75 0.75 1.0"/>
+		      </material>
+		    </visual>
+		    <collision>
+		      <origin rpy="0 0 0" xyz="0 0 0"/>
+		      <geometry>
+			<mesh filename="package://igor/meshes/finger_prox_link_simple.dae" scale="0.5 0.5 0.5"/>
 		      </geometry>
 		      <material name="light_grey">
@@ -547,14 +547,14 @@
 		      <origin rpy="0 0 0" xyz="0 0 0"/>
 		      <geometry>
-			<mesh filename="package://fh_desc/meshes/v2/finger_dist_link_simple.dae" scale="0.5 0.5 0.5"/>
-		      </geometry>
-		      <material name="light_grey">
-			<color rgba="0.75 0.75 0.75 1.0"/>
-		      </material>
-		    </visual>
-		    <collision>
-		      <origin rpy="0 0 0" xyz="0 0 0"/>
-		      <geometry>
-			<mesh filename="package://fh_desc/meshes/v2/finger_dist_link_simple.dae" scale="0.5 0.5 0.5"/>
+			<mesh filename="package://igor/meshes/finger_dist_link_simple.dae" scale="0.5 0.5 0.5"/>
+		      </geometry>
+		      <material name="light_grey">
+			<color rgba="0.75 0.75 0.75 1.0"/>
+		      </material>
+		    </visual>
+		    <collision>
+		      <origin rpy="0 0 0" xyz="0 0 0"/>
+		      <geometry>
+			<mesh filename="package://igor/meshes/finger_dist_link_simple.dae" scale="0.5 0.5 0.5"/>
 		      </geometry>
 		      <material name="light_grey">
@@ -629,14 +629,14 @@
 		      <origin rpy="0 0 0" xyz="0 0 0"/>
 		      <geometry>
-			<mesh filename="package://fh_desc/meshes/omd-d18-tip.dae" scale="0.5 0.5 0.5"/>
-		      </geometry>
-		      <material name="light_grey">
-			<color rgba="0.75 0.75 0.75 1.0"/>
-		      </material>
-		    </visual>
-		    <collision>
-		      <origin rpy="0 0 0" xyz="0 0 0"/>
-		      <geometry>
-			<mesh filename="package://fh_desc/meshes/omd-d18-tip.dae" scale="0.5 0.5 0.5"/>
+			<mesh filename="package://igor/meshes/omd-d18-tip.dae" scale="0.5 0.5 0.5"/>
+		      </geometry>
+		      <material name="light_grey">
+			<color rgba="0.75 0.75 0.75 1.0"/>
+		      </material>
+		    </visual>
+		    <collision>
+		      <origin rpy="0 0 0" xyz="0 0 0"/>
+		      <geometry>
+			<mesh filename="package://igor/meshes/omd-d18-tip.dae" scale="0.5 0.5 0.5"/>
 		      </geometry>
 		      <material name="light_grey">

Commit message: SG filter Python file added

File: urdf/Igor_armed.urdf.xacro (robot description, xacro)
@@ -127,5 +127,5 @@
 		<origin xyz="${0} ${0} ${base_z_size/2 + 0.015}" rpy="${M_PI/2} 0 0" />
 	</xacro:igor_actuator>
-	<xacro:arm prefix="Upper" reflect="-1" flip="0">
+	<xacro:arm prefix="Upper" reflect="-1" flip="0" lower_limit="-3" upper_limit="3">
 		<origin xyz="${0} ${actuator_y_size/2+lower_leg_radius} ${0.0}" rpy="${-M_PI/2} ${0} ${0}" />
 	</xacro:arm>
@@ -134,5 +134,5 @@
 		<origin xyz="${lower_leg_length + actuator_z_size/2.3} ${0} -${actuator_y_size/1.2}" rpy="${M_PI/2} ${0} 0" />
 	</xacro:igor_actuator>
-	<xacro:arm prefix="Fore" reflect="1" flip="1">
+	<xacro:arm prefix="Fore" reflect="1" flip="1" lower_limit="-2.5" upper_limit="2.5">
 		<origin xyz="${0} -${actuator_y_size/2+lower_leg_radius} 0.0" rpy="${-M_PI/2} ${0} ${0}" />
 	</xacro:arm>

File: urdf/arm.urdf.xacro (robot description, xacro)
@@ -1,5 +1,5 @@
 <?xml version="1.0"?>
 <robot xmlns:xacro="http://ros.org/wiki/xacro" name="arm">
-	<xacro:macro name="arm" params="prefix reflect flip *joint_pose">
+	<xacro:macro name="arm" params="prefix reflect flip lower_limit upper_limit *joint_pose">
 		<link name="${prefix}_arm">
 			<visual>
@@ -26,5 +26,5 @@
 			<parent link="${prefix}_armActuator"/>
 			<child  link="${prefix}_arm"/>
-			<limit effort="25" lower="${-2}" upper="${2}" velocity="10"/>
+			<limit effort="15" lower="${lower_limit}" upper="${upper_limit}" velocity="15"/>
 			<axis xyz="0 0 1"/>
 			<dynamics damping="0.1"/>

File: urdf/pepsi_can.urdf.xacro (robot description, xacro)
@@ -18,5 +18,5 @@
 	    		<inertial>
 				<origin rpy="${0} ${0} ${0}" xyz="${0} ${0} ${0}"/>
-	      			<mass value="0.241"/>
+	      			<mass value="${0.241*1.5}"/>
 	      			<inertia ixx="${0.00038433}" ixy="0.00" ixz="0.00" izz="${0.000170013}" iyz="0.000" iyy="0.00038433"/>
 	    		</inertial>

Commit message: Update

File: urdf/Igor_armed.urdf.xacro (robot description, xacro)
@@ -181,5 +181,5 @@
 		<plugin name="p3d_base_controller" filename= "libgazebo_ros_p3d.so">
 			<robotNamespace>/igor</robotNamespace>
-			<alwaysOn>true</alwaysOn>
+			<alwaysOn>false</alwaysOn>
 			<updateRate>500.0</updateRate>
 			<bodyName>base_link</bodyName>
@@ -195,5 +195,5 @@
 		<plugin name="p3d_base_controller" filename= "libgazebo_ros_p3d.so">
 			<robotNamespace>/igor</robotNamespace>
-			<alwaysOn>true</alwaysOn>
+			<alwaysOn>false</alwaysOn>
 			<updateRate>500.0</updateRate>
 			<bodyName>robot_center_link</bodyName>
@@ -209,5 +209,5 @@
 	    <gravity>true</gravity>
 	    <sensor name="body_imu" type="imu">
-	      <always_on>true</always_on>
+	      <always_on>false</always_on>
 	      <visualize>true</visualize>
 	      <!--topic>__default_topic__</topic-->

File: urdf/pepsi_can.urdf.xacro (robot description, xacro)
@@ -18,6 +18,6 @@
 	    		<inertial>
 				<origin rpy="${0} ${0} ${0}" xyz="${0} ${0} ${0}"/>
-	      			<mass value="${0.241*1.5}"/>
-	      			<inertia ixx="${0.00038433}" ixy="0.00" ixz="0.00" izz="${0.000170013}" iyz="0.000" iyy="0.00038433"/>
+	      			<mass value="${0.241*3}"/>
+	      			<inertia ixx="${0.00038433*3}" ixy="0.00" ixz="0.00" izz="${0.000170013*3}" iyz="0.000" iyy="${0.00038433*3}"/>
 	    		</inertial>
 	    	</link>
