Commit message: L1 Adaptive for HW ver.1

File: urdf/Igor_armed.urdf.xacro (robot description, xacro)
@@ -127,5 +127,5 @@
 		<origin xyz="${0} ${0} ${base_z_size/2 + 0.015}" rpy="${M_PI/2} 0 0" />
 	</xacro:igor_actuator>
-	<xacro:arm prefix="Upper" reflect="-1" flip="0" lower_limit="-3" upper_limit="3">
+	<xacro:arm prefix="Upper" reflect="-1" flip="0" lower_limit="0.78" upper_limit="0.78">
 		<origin xyz="${0} ${actuator_y_size/2+lower_leg_radius} ${0.0}" rpy="${-M_PI/2} ${0} ${0}" />
 	</xacro:arm>
@@ -134,5 +134,5 @@
 		<origin xyz="${lower_leg_length + actuator_z_size/2.3} ${0} -${actuator_y_size/1.2}" rpy="${M_PI/2} ${0} 0" />
 	</xacro:igor_actuator>
-	<xacro:arm prefix="Fore" reflect="1" flip="1" lower_limit="-2.5" upper_limit="2.5">
+	<xacro:arm prefix="Fore" reflect="1" flip="1" lower_limit="-1.5708" upper_limit="-1.5708">
 		<origin xyz="${0} -${actuator_y_size/2+lower_leg_radius} 0.0" rpy="${-M_PI/2} ${0} ${0}" />
 	</xacro:arm>
@@ -146,7 +146,7 @@
 	</xacro:my_hand>
 	<!--Pepsi Can  -->
-	<xacro:pepsi_can parent_link= "H1_base_link">
+	<!--xacro:pepsi_can parent_link= "H1_base_link">
 		<origin xyz="${0.0} ${0} ${0.062}" rpy="${0} ${0} ${0}" />
-	</xacro:pepsi_can>
+	</xacro:pepsi_can-->
 	<!--Robot Center Dummy-->
 	<link name="robot_center_link">

File: urdf/Igor_knee.urdf.xacro (robot description, xacro)
@@ -46,6 +46,6 @@
 		<!--inertial>
      			<origin xyz="0 0 0" rpy="0.0 0.0 0.0" />
-			<mass value="4" />
-      			<inertia izz="0.036344" iyz="0.0" ixz="0.00" iyy="0.036344" ixy="0.000" ixx="0.061936" />
+			<mass value="${5}" />
+      			<inertia izz="${0.04543}" iyz="0.0" ixz="0.00" iyy="${0.04543}" ixy="0.000" ixx="${0.0774}" />
 		</inertial-->
 		<visual>
@@ -117,5 +117,5 @@
 		<origin xyz="${0} -${actuator_y_size-0.0038} -${lower_leg_length+actuator_z_size/2.5}" rpy="0 0 0" />
 	</xacro:igor_actuator>
-	<xacro:igor_wheel prefix="R" flip="0" reflect="-1" damping="${0.17}" static_friction="0.0011">
+	<xacro:igor_wheel prefix="R" flip="0" reflect="-1" damping="${1*0.17}" static_friction="0.0011">
 		<origin xyz="${0} -${(actuator_y_size/2)+wheel_length/2} 0.0" rpy="0 0 0" />
 	</xacro:igor_wheel>
@@ -124,5 +124,5 @@
 		<origin xyz="${0} ${actuator_y_size-0.0038} -${lower_leg_length+actuator_z_size/2.5}" rpy="0 0 0" />
 	</xacro:igor_actuator>
-	<xacro:igor_wheel prefix="L" flip="1" reflect="1" damping="${0.17}" static_friction="0.0011">
+	<xacro:igor_wheel prefix="L" flip="1" reflect="1" damping="${1*0.17}" static_friction="0.0011">
 		<origin xyz="${0} ${(actuator_y_size/2)+wheel_length/2} 0.0" rpy="0 0 0" />
 	</xacro:igor_wheel>
