Commit message: L1 controller added

File: urdf/pepsi_can.urdf.xacro (robot description, xacro)
@@ -18,6 +18,6 @@
 	    		<inertial>
 				<origin rpy="${0} ${0} ${0}" xyz="${0} ${0} ${0}"/>
-	      			<mass value="${0.241*3}"/>
-	      			<inertia ixx="${0.00038433*3}" ixy="0.00" ixz="0.00" izz="${0.000170013*3}" iyz="0.000" iyy="${0.00038433*3}"/>
+	      			<mass value="${0.241*1.5}"/>
+	      			<inertia ixx="${0.00038433}" ixy="0.00" ixz="0.00" izz="${0.000170013}" iyz="0.000" iyy="${0.00038433}"/>
 	    		</inertial>
 	    	</link>
