Commit message: Updated

File: urdf/wheel.urdf.xacro (robot description, xacro)
@@ -39,5 +39,5 @@
 			<parent link="${prefix}_wheelActuator"/>
 			<child  link="${prefix}_wheel"/>
-			<limit effort="3" velocity="12"/>  <!-- effort limit in N (prismatic) or N.m (revolute), Velocity limit in m/s or rad/s -->
+			<limit effort="5" velocity="20"/>  <!-- effort limit in N (prismatic) or N.m (revolute), Velocity limit in m/s or rad/s -->
 			<axis xyz="0 1 0"/>
 			<dynamics damping="${damping}" friction="${static_friction}"/>

Commit message: L1 1DoF functional

File: urdf/wheel.urdf.xacro (robot description, xacro)
@@ -39,5 +39,5 @@
 			<parent link="${prefix}_wheelActuator"/>
 			<child  link="${prefix}_wheel"/>
-			<limit effort="5" velocity="20"/>  <!-- effort limit in N (prismatic) or N.m (revolute), Velocity limit in m/s or rad/s -->
+			<limit effort="500" velocity="50"/>  <!-- effort limit in N (prismatic) or N.m (revolute), Velocity limit in m/s or rad/s -->
 			<axis xyz="0 1 0"/>
 			<dynamics damping="${damping}" friction="${static_friction}"/>

Commit message: L1 Controller SISO Ver.2

File: urdf/wheel.urdf.xacro (robot description, xacro)
@@ -39,5 +39,5 @@
 			<parent link="${prefix}_wheelActuator"/>
 			<child  link="${prefix}_wheel"/>
-			<limit effort="500" velocity="50"/>  <!-- effort limit in N (prismatic) or N.m (revolute), Velocity limit in m/s or rad/s -->
+			<limit effort="5" velocity="20"/>  <!-- effort limit in N (prismatic) or N.m (revolute), Velocity limit in m/s or rad/s -->
 			<axis xyz="0 1 0"/>
 			<dynamics damping="${damping}" friction="${static_friction}"/>
